File: Hardware/Qwiic Shield for RaspberryPi.brd (EAGLE design)
At the start: 52.3 x 23 mm, 22 parts, among them J1 Qwiic Right Angle, J6 Qwiic Right Angle, J7 Qwiic Right Angle, J8 Qwiic Right Angle, U2 3.3V/600mA, U3 RASPBERRY_PI

Commit message: Engineering checklist changes
Routing:
- net D12: track 8.95 -> 8.39 mm
Changed lines of the file:
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@@
 <layer number="20" name="Dimension" color="15" fill="1" visible="yes" active="yes"/>
 <layer number="21" name="tPlace" color="16" fill="1" visible="yes" active="yes"/>
-<layer number="22" name="bPlace" color="14" fill="1" visible="yes" active="yes"/>
+<layer number="22" name="bPlace" color="14" fill="1" visible="no" active="yes"/>
 <layer number="23" name="tOrigins" color="15" fill="1" visible="yes" active="yes"/>
 <layer number="24" name="bOrigins" color="15" fill="1" visible="yes" active="yes"/>
@@
 <text x="48.641" y="0.508" size="1.27" layer="16" font="vector" ratio="15" rot="MR0">v01</text>
 <text x="21.59" y="-26.67" size="1.778" layer="51" font="vector">A. England</text>
+<dimension x1="0" y1="0" x2="0" y2="22.86" x3="-8.89" y3="11.43" textsize="1.778" layer="47" unit="inch"/>
+<dimension x1="52.07" y1="0" x2="0" y2="0" x3="26.035" y3="-5.08" textsize="1.778" layer="47" unit="inch"/>
 </plain>
 <attributes>
@@
 <contactref element="U3" pad="32"/>
 <contactref element="J4" pad="2"/>
-<wire x1="36.83" y1="8.89" x2="36.83" y2="12.7" width="0.1778" layer="1"/>
-<wire x1="36.83" y1="12.7" x2="38.862" y2="14.732" width="0.1778" layer="1"/>
-<wire x1="40.12" y1="15.905" x2="39.146" y2="15.905" width="0.1778" layer="1"/>
-<wire x1="39.146" y1="15.905" x2="38.862" y2="15.621" width="0.1778" layer="1"/>
-<wire x1="38.862" y1="15.621" x2="38.862" y2="14.732" width="0.1778" layer="1"/>
+<wire x1="36.83" y1="8.89" x2="36.83" y2="10.922" width="0.2032" layer="1"/>
+<wire x1="36.83" y1="10.922" x2="40.132" y2="14.224" width="0.1778" layer="1"/>
+<wire x1="40.132" y1="14.224" x2="40.132" y2="15.893" width="0.1778" layer="1"/>
+<wire x1="40.132" y1="15.893" x2="40.12" y2="15.905" width="0.2032" layer="1"/>
 </signal>
 <signal name="D13">

Commit message: Post design review changes
Parts:
- moved FD1 2.84 mm to (1.27, 12.7)
- moved FD4 2.84 mm to (1.27, 12.7)
Routing:
- net 5V: track 21.5 -> 23.4 mm
Changed lines of the file:
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@@
 <element name="FRAME1" library="SparkFun-Aesthetics" package="CREATIVE_COMMONS" value="FRAME-LETTER" x="-8.89" y="-24.13"/>
 <element name="LOGO1" library="SparkFun-Aesthetics" package="OSHW-LOGO-MINI" value="OSHW-LOGOMINI" x="7.493" y="6.096"/>
-<element name="FD1" library="SparkFun-Aesthetics" package="FIDUCIAL-1X2" value="FIDUCIAL1X2" x="3.81" y="13.97" rot="R180"/>
+<element name="FD1" library="SparkFun-Aesthetics" package="FIDUCIAL-1X2" value="FIDUCIAL1X2" x="1.27" y="12.7" rot="R180"/>
 <element name="FD2" library="SparkFun-Aesthetics" package="FIDUCIAL-1X2" value="FIDUCIAL1X2" x="50.8" y="2.54" rot="R180"/>
 <element name="J1" library="SparkFun-Connectors" package="1X04_1MM_RA" value="Qwiic Right Angle" x="39.37078125" y="5.08011875">
@@
 </element>
 <element name="FD3" library="SparkFun-Aesthetics" package="FIDUCIAL-1X2" value="FIDUCIAL1X2" x="50.8" y="2.54" rot="MR0"/>
-<element name="FD4" library="SparkFun-Aesthetics" package="FIDUCIAL-1X2" value="FIDUCIAL1X2" x="3.81" y="13.97" rot="MR0"/>
+<element name="FD4" library="SparkFun-Aesthetics" package="FIDUCIAL-1X2" value="FIDUCIAL1X2" x="1.27" y="12.7" rot="MR0"/>
 <element name="LOGO2" library="SparkFun-Aesthetics" package="REVISION" value="REVISION" x="2.54" y="-26.67"/>
 </elements>
@@
 <contactref element="U2" pad="1"/>
 <contactref element="U2" pad="3"/>
-<wire x1="2.02" y1="15.905" x2="2.02" y2="8.89" width="0.3048" layer="1"/>
 <wire x1="2.02" y1="8.89" x2="2.02" y2="6.35" width="0.3048" layer="1"/>
 <wire x1="2.02" y1="6.35" x2="2.02" y2="5.473" width="0.3048" layer="1"/>
@@
 <wire x1="3.241" y1="3.49" x2="3.429" y2="3.302" width="0.3048" layer="1"/>
 <wire x1="3.429" y1="3.302" x2="3.429" y2="1.651" width="0.3048" layer="1"/>
-<wire x1="3.81" y1="8.89" x2="2.02" y2="8.89" width="0.3048" layer="1"/>
-<wire x1="4.56" y1="15.905" x2="2.02" y2="15.905" width="0.3048" layer="1"/>
+<wire x1="3.81" y1="8.89" x2="2.032" y2="8.89" width="0.3048" layer="1"/>
 <wire x1="2.96" y1="6.35" x2="2.02" y2="6.35" width="0.3048" layer="1"/>
+<wire x1="2.02" y1="8.89" x2="2.032" y2="8.89" width="0.3048" layer="1"/>
+<wire x1="2.032" y1="8.89" x2="2.032" y2="10.795" width="0.3048" layer="1"/>
+<wire x1="2.032" y1="10.795" x2="3.302" y2="12.065" width="0.3048" layer="1"/>
+<wire x1="3.302" y1="12.065" x2="3.302" y2="13.97" width="0.3048" layer="1"/>
+<wire x1="2.02" y1="15.905" x2="2.02" y2="14.49" width="0.3048" layer="1"/>
+<wire x1="2.02" y1="14.49" x2="2.54" y2="13.97" width="0.3048" layer="1"/>
+<wire x1="2.54" y1="13.97" x2="3.302" y2="13.97" width="0.3048" layer="1"/>
+<wire x1="3.302" y1="13.97" x2="4.191" y2="13.97" width="0.3048" layer="1"/>
+<wire x1="4.191" y1="13.97" x2="4.572" y2="14.351" width="0.3048" layer="1"/>
+<wire x1="4.572" y1="14.351" x2="4.572" y2="15.893" width="0.3048" layer="1"/>
+<wire x1="4.572" y1="15.893" x2="4.56" y2="15.905" width="0.3048" layer="1"/>
 </signal>
 <signal name="RX">
