File: Hardware/Qwiic_pHat_for_Raspberry_Pi_v30.brd (EAGLE design)
At the start: 65 x 30.5 mm, 44 parts, among them J1 RASPBERRYPI-40-PIN-GPIO_PTH_N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, J4 Qwiic Right Angle, J7 Qwiic Right Angle

Commit message: Swaps power and ground on screw terminal, adjusts silk in various areas
Parts:
- added U$17: (no value), SparkFun-Aesthetics:QWIIC_3MM
- added U$18: (no value), Qwiic:QWIIC0
- LOGO3: value SFE_LOGO_NAME_FLAME.1_INCH -> SFE_LOGO_NAME.1_INCH; device SparkFun-Aesthetics:SFE_LOGO_NAME_FLAME_.1 -> SparkFun-Aesthetics:SFE_LOGO_NAME_.1
- U$1: device Qwiic:QWIIC1 -> pie_1f967#png:PIE_1F967#PNG
- U$8: device All labels:BUTTON2 -> SparkFun-Aesthetics:QWIIC_3MM
- moved U$1 25.7 mm to (34.8, 22.1), turned to 20 degrees
- moved U$8 6.60 mm to (39.4, 17.8)
- moved U$9 1.52 mm to (45.5, 15.2)
- moved U$10 1.06 mm to (33.5, 11.4)
- moved LOGO3 0.23 mm to (33.0, 19.8)
Connections:
- net 5V: now also J2.2, J3.2; no longer J2.1, J3.1
- net GND: now also J2.1, J3.1; no longer J2.2, J3.2
Routing:
- net 5V: track 12.1 -> 13.5 mm, vias 0 -> 1
Changed lines of the file:
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@@
 <drawing>
 <settings>
-<setting alwaysvectorfont="yes"/>
+<setting alwaysvectorfont="no"/>
 <setting keepoldvectorfont="yes"/>
 <setting verticaltext="up"/>
 </settings>
-<grid distance="0.01" unitdist="inch" unit="mm" style="lines" multiple="1" display="yes" altdistance="0.001" altunitdist="inch" altunit="mm"/>
+<grid distance="0.01" unitdist="inch" unit="inch" style="lines" multiple="1" display="yes" altdistance="0.001" altunitdist="inch" altunit="inch"/>
 <layers>
 <layer number="1" name="Top" color="4" fill="1" visible="yes" active="yes"/>
@@
 <dimension x1="0" y1="0.000003125" x2="65" y2="0" x3="32.5" y3="-8.999996875" textsize="1.778" textratio="15" layer="47"/>
 <dimension x1="3.5" y1="3.5" x2="0" y2="3.4798" x3="1.799315625" y3="-5.05495625" textsize="1.778" textratio="15" layer="47"/>
-<text x="10.3632" y="17.9324" size="2.286" layer="21" font="vector" ratio="15">+</text>
-<text x="10.414" y="14.3764" size="2.286" layer="21" font="vector" ratio="15">-</text>
-<text x="12.065" y="14.3764" size="2.286" layer="22" font="vector" ratio="15" rot="MR0">-</text>
-<text x="12.0142" y="17.9324" size="2.286" layer="22" font="vector" ratio="15" rot="MR0">+</text>
+<text x="10.3632" y="14.3764" size="2.286" layer="21" font="vector" ratio="15">+</text>
+<text x="10.414" y="17.9324" size="2.286" layer="21" font="vector" ratio="15">-</text>
+<text x="12.065" y="17.9324" size="2.286" layer="22" font="vector" ratio="15" rot="MR0">-</text>
+<text x="12.0142" y="14.3764" size="2.286" layer="22" font="vector" ratio="15" rot="MR0">+</text>
 </plain>
 <attributes>
@@
 <attribute name="VALUE" x="42.8056" y="3.5" size="0.6096" layer="27" font="vector" ratio="20" rot="R90" align="top-center"/>
 </element>
-<element name="LOGO3" library="SparkFun-Aesthetics" package="SFE_LOGO_NAME_FLAME_.1" value="SFE_LOGO_NAME_FLAME.1_INCH" x="32.806" y="19.9" smashed="yes"/>
 <element name="LOGO2" library="SparkFun-Aesthetics" package="OSHW-LOGO-S" value="OSHW-LOGOS" x="32.386" y="2.222" smashed="yes"/>
 <element name="U$3" library="MicroPiHat" package="PHAT0" value="" x="30.294" y="9.238" smashed="yes"/>
@@
 <attribute name="VALUE" x="10.16" y="20.32" size="0.6096" layer="27" font="vector" ratio="20" rot="R270"/>
 </element>
-<element name="U$8" library="All labels" package="BUTTON2" value="" x="45.466" y="15.24" smashed="yes"/>
-<element name="U$9" library="All labels" package="GPIO173" value="" x="45.466" y="13.716" smashed="yes"/>
-<element name="U$10" library="SparkFun-Aesthetics" package="SFE_LOGO_NAME_FLAME_.3" value="" x="32.5" y="11.684" smashed="yes" rot="MR0"/>
+<element name="U$9" library="All labels" package="GPIO173" value="" x="45.466" y="15.24" smashed="yes"/>
 <element name="F1" library="SparkFun-Fuses" package="1206" value="6V/0.75A" x="6.35" y="22.098" smashed="yes">
 <attribute name="NAME" x="6.35" y="23.241" size="0.6096" layer="25" font="vector" ratio="20" align="bottom-center"/>
@@
 <element name="U$6" library="Fuse Bypass" package="FUSE0" value="" x="14.224" y="22.606" smashed="yes" rot="MR0"/>
 <element name="U$7" library="Fuse Bypass" package="BYPASS1" value="" x="16.256" y="21.082" smashed="yes" rot="MR0"/>
-<element name="U$1" library="Qwiic" package="QWIIC1" value="" x="12.7" y="8.89" smashed="yes"/>
 <element name="U$11" library="SparkFun-Aesthetics" package="QWIIC_3MM" value="" x="62.992" y="23.368" smashed="yes"/>
 <element name="U$12" library="POWER" package="5V0" value="" x="-1.016" y="12.446" smashed="yes"/>
@@
 <element name="U$15" library="POWER" package="5V0" value="" x="5.334" y="12.446" smashed="yes" rot="MR0"/>
 <element name="U$16" library="SparkFun-Aesthetics" package="QWIIC_3MM" value="" x="63.246" y="14.732" smashed="yes"/>
+<element name="U$8" library="SparkFun-Aesthetics" package="QWIIC_3MM" value="" x="39.37" y="17.78" smashed="yes"/>
+<element name="U$17" library="SparkFun-Aesthetics" package="QWIIC_3MM" value="" x="25.908" y="17.78" smashed="yes"/>
+<element name="U$18" library="Qwiic" package="QWIIC0" value="" x="13.208" y="8.89" smashed="yes"/>
+<element name="U$1" library="pie_1f967#png" package="PIE_1F967#PNG" value="" x="34.798" y="22.098" smashed="yes" rot="R20"/>
+<element name="LOGO3" library="SparkFun-Aesthetics" package="SFE_LOGO_NAME_.1" value="SFE_LOGO_NAME.1_INCH" x="33.02" y="19.812" smashed="yes"/>
+<element name="U$10" library="SparkFun-Aesthetics" package="SFE_LOGO_NAME_FLAME_.3" value="" x="33.528" y="11.43" smashed="yes" rot="MR0"/>
 </elements>
 <signals>
@@
 <via x="32.811" y="6.954" extent="1-16" drill="0.508"/>
 <via x="54.67" y="10.645" extent="1-16" drill="0.508"/>
-<contactref element="J3" pad="2"/>
 <contactref element="S1" pad="1"/>
 <contactref element="J6" pad="1"/>
 <contactref element="J5" pad="1"/>
-<contactref element="J2" pad="2"/>
+<contactref element="J3" pad="1"/>
+<contactref element="J2" pad="1"/>
 </signal>
 <signal name="3.3V">
@@
 </signal>
 <signal name="5V">
-<contactref element="J3" pad="1"/>
-<contactref element="J2" pad="1"/>
-<wire x1="8.89" y1="19.05" x2="6.604" y2="19.05" width="0.508" layer="1"/>
 <contactref element="F1" pad="2"/>
-<wire x1="6.604" y1="19.05" x2="3.81" y2="19.05" width="0.508" layer="1"/>
 <wire x1="7.75" y1="22.098" x2="7.75" y2="21.847" width="0.508" layer="1"/>
 <wire x1="7.75" y1="21.847" x2="6.604" y2="20.701" width="0.508" layer="1"/>
-<wire x1="6.604" y1="20.701" x2="6.604" y2="19.05" width="0.508" layer="1"/>
 <contactref element="JP1" pad="2"/>
 <wire x1="6.2738" y1="21.5646" x2="6.2738" y2="21.5138" width="0.508" layer="16"/>
-<wire x1="6.2738" y1="21.5138" x2="3.81" y2="19.05" width="0.508" layer="16"/>
+<contactref element="J3" pad="2"/>
+<contactref element="J2" pad="2"/>
+<wire x1="3.81" y1="15.55" x2="6.604" y2="15.55" width="0.508" layer="1"/>
+<wire x1="6.604" y1="15.55" x2="8.89" y2="15.55" width="0.508" layer="1"/>
+<wire x1="6.604" y1="20.701" x2="6.604" y2="20.32" width="0.508" layer="1"/>
+<wire x1="6.604" y1="20.32" x2="6.604" y2="15.55" width="0.508" layer="1"/>
+<wire x1="6.2738" y1="21.5646" x2="6.2738" y2="20.6502" width="0.508" layer="16"/>
+<wire x1="6.2738" y1="20.6502" x2="6.604" y2="20.32" width="0.508" layer="16"/>
+<via x="6.604" y="20.32" extent="1-16" drill="0.508"/>
 </signal>
 <signal name="RX">
