File: Hardware/Qwiic_pHat_for_Raspberry_Pi_v30.brd (EAGLE design)
At the start: 65 x 30.5 mm, 44 parts, among them J1 RASPBERRYPI-40-PIN-GPIO_PTH_N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, J4 Qwiic Right Angle, J5 Vertical Qwiic Connector, J6 Vertical Qwiic Connector, J7 Qwiic Right Angle

Commit message: Update Qwiic_pHat_for_Raspberry_Pi_v30.brd
- Adjust Measures Layer for Board/Mounting Hole Dimensions
- Make Text Ratio the Uniform for Measures
- Move Aesthetics Down to Read Measures Layer
Parts:
- moved FRAME1 8.90 mm to (-1.02, -21.8)
- moved LOGO1 8.90 mm to (10.4, -24.4)
Changed lines of the file:
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@@
 <?xml version="1.0" encoding="utf-8"?>
 <!DOCTYPE eagle SYSTEM "eagle.dtd">
-<eagle version="9.4.2">
+<eagle version="9.5.0">
 <drawing>
 <settings>
@@
 <layer number="45" name="Holes" color="7" fill="1" visible="yes" active="yes"/>
 <layer number="46" name="Milling" color="3" fill="1" visible="no" active="yes"/>
-<layer number="47" name="Measures" color="7" fill="1" visible="no" active="yes"/>
+<layer number="47" name="Measures" color="7" fill="1" visible="yes" active="yes"/>
 <layer number="48" name="Document" color="7" fill="1" visible="no" active="yes"/>
 <layer number="49" name="Reference" color="13" fill="1" visible="yes" active="yes"/>
@@
 <wire x1="0" y1="27.5" x2="0" y2="3" width="0.2032" layer="20"/>
 <wire x1="0" y1="3" x2="3" y2="0" width="0.2032" layer="20" curve="90"/>
-<text x="30.226" y="-12.954" size="1.778" layer="51" font="vector">N. Seidle</text>
+<text x="30.734" y="-21.844" size="1.778" layer="51" font="vector">N. Seidle</text>
 <text x="55.771" y="0.818" size="1.27" layer="16" font="vector" ratio="15" rot="MR0">v30</text>
-<text x="28.956" y="-15.494" size="1.778" layer="51" font="vector">A. England and Elias Santistevan</text>
-<dimension x1="0" y1="30.5" x2="0" y2="0" x3="-5" y3="15.25" textsize="1.778" layer="47"/>
-<dimension x1="3.5" y1="26.5" x2="32.5" y2="26.5" x3="18" y3="32.5" textsize="1.778" layer="47"/>
-<dimension x1="3.5" y1="26.5" x2="61.5" y2="26.5" x3="32.5" y3="37" textsize="1.778" layer="47"/>
+<text x="29.464" y="-24.384" size="1.778" layer="51" font="vector">A. England and Elias Santistevan</text>
+<dimension x1="0" y1="30.5" x2="0" y2="0" x3="-5" y3="15.25" textsize="1.778" textratio="15" layer="47"/>
+<dimension x1="3.5" y1="26.5" x2="32.5" y2="26.5" x3="18" y3="32.5" textsize="1.778" textratio="15" layer="47"/>
+<dimension x1="3.5" y1="26.5" x2="61.5" y2="26.5" x3="32.5" y3="37" textsize="1.778" textratio="15" layer="47"/>
 <circle x="3.5" y="3.5" radius="3.15" width="0" layer="41"/>
 <circle x="61.5" y="3.5" radius="3.15" width="0" layer="41"/>
@@
 <circle x="41.19" y="3.49" radius="3.15" width="0" layer="41"/>
 <circle x="23.88" y="3.5" radius="3.15" width="0" layer="41"/>
-<text x="21" y="-13" size="2" layer="47" font="vector">Units in MM</text>
+<text x="21.508" y="-12.746" size="2" layer="47" font="vector">Units in MM</text>
 <dimension x1="3.5" y1="3.5" x2="3.5" y2="26.5" x3="-2" y3="15" textsize="1.778" textratio="15" layer="47"/>
-<dimension x1="36.1" y1="3.5" x2="61.5" y2="3.5" x3="48.8" y3="-3.81" textsize="1.778" textratio="15" layer="47"/>
 <dimension x1="0" y1="0.000003125" x2="65" y2="0" x3="32.5" y3="-8.999996875" textsize="1.778" textratio="15" layer="47"/>
-<dimension x1="3.5" y1="3.5" x2="0" y2="3.4798" x3="1.799315625" y3="-5.05495625" textsize="1.778" textratio="15" layer="47"/>
 <text x="10.3632" y="14.3764" size="2.286" layer="21" font="vector" ratio="15">+</text>
 <text x="10.414" y="17.9324" size="2.286" layer="21" font="vector" ratio="15">-</text>
 <text x="12.065" y="17.9324" size="2.286" layer="22" font="vector" ratio="15" rot="MR0">-</text>
 <text x="12.0142" y="14.3764" size="2.286" layer="22" font="vector" ratio="15" rot="MR0">+</text>
+<dimension x1="61.5" y1="3.5" x2="41.1546" y2="3.5" x3="51.3273" y3="-3.556" textsize="1.778" textratio="15" layer="47"/>
+<dimension x1="3.5" y1="3.5" x2="0" y2="3.302" x3="1.75" y3="-3.81" textsize="1.778" textratio="15" layer="47" dtype="horizontal"/>
 </plain>
 <attributes>
@@
 </autorouter>
 <elements>
-<element name="FRAME1" library="SparkFun-Aesthetics" package="CREATIVE_COMMONS" value="FRAME-LETTER" x="-1.524" y="-12.954" smashed="yes">
-<attribute name="DESIGNER" value="" x="-1.524" y="-12.954" size="1.778" layer="27" display="off"/>
-<attribute name="REV" value="" x="-1.524" y="-12.954" size="1.778" layer="27" display="off"/>
+<element name="FRAME1" library="SparkFun-Aesthetics" package="CREATIVE_COMMONS" value="FRAME-LETTER" x="-1.016" y="-21.844" smashed="yes">
+<attribute name="DESIGNER" value="" x="-1.016" y="-21.844" size="1.778" layer="27" display="off"/>
+<attribute name="REV" value="" x="-1.016" y="-21.844" size="1.778" layer="27" display="off"/>
 </element>
 <element name="FD1" library="SparkFun-Aesthetics" package="FIDUCIAL-1X2" value="FIDUCIAL1X2" x="6.52" y="29.56" smashed="yes" rot="R180"/>
@@
 <element name="FD3" library="SparkFun-Aesthetics" package="FIDUCIAL-1X2" value="FIDUCIAL1X2" x="57.33" y="1.31" smashed="yes" rot="MR0"/>
 <element name="FD4" library="SparkFun-Aesthetics" package="FIDUCIAL-1X2" value="FIDUCIAL1X2" x="6.52" y="29.56" smashed="yes" rot="MR0"/>
-<element name="LOGO1" library="SparkFun-Aesthetics" package="REVISION" value="REVISION" x="9.906" y="-15.494" smashed="yes"/>
+<element name="LOGO1" library="SparkFun-Aesthetics" package="REVISION" value="REVISION" x="10.414" y="-24.384" smashed="yes"/>
 <element name="J1" library="SparkFun-Connectors" package="2X20" value="RASPBERRYPI-40-PIN-GPIO_PTH_NO_SHROUD" x="8.37" y="25.2" smashed="yes">
 <attribute name="NAME" x="7.1" y="29.264" size="0.6096" layer="25" font="vector" ratio="20"/>
