File: Hardware/Qwiic_pHat_for_Raspberry_Pi_v30.sch (EAGLE design)
At the start: 28 parts, among them J1 RASPBERRYPI-40-PIN-GPIO_PTH_N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, J4 Qwiic Right Angle, J7 Qwiic Right Angle

Commit message: Updates Vertical Qwiic connector to have value of "vertical qwiic connector"
Parts:
- J5, J6: value (none) -> Vertical Qwiic Connector
Changed lines of the file:
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@@
 <part name="R3" library="SparkFun-Resistors" deviceset="10KOHM" device="-0603-1/10W-1%" value="10k"/>
 <part name="SUPPLY7" library="SparkFun-PowerSymbols" deviceset="3.3V" device=""/>
-<part name="J5" library="SparkFun-Connectors" deviceset="QWIIC_CONNECTOR" device=""/>
-<part name="J6" library="SparkFun-Connectors" deviceset="QWIIC_CONNECTOR" device=""/>
 <part name="GND5" library="SparkFun-PowerSymbols" deviceset="GND" device=""/>
 <part name="SUPPLY6" library="SparkFun-PowerSymbols" deviceset="3.3V" device=""/>
@@
 <part name="JP1" library="SparkFun-Jumpers" deviceset="JUMPER-SMT_2_NO" device="_SILK" value="JUMPER-SMT_2_NO_SILK"/>
 <part name="LOGO3" library="SparkFun-Aesthetics" deviceset="SFE_LOGO_NAME" device=".1_INCH" value="SFE_LOGO_NAME.1_INCH"/>
+<part name="J5" library="SparkFun-Connectors" deviceset="QWIIC_CONNECTOR" device="" value="Vertical Qwiic Connector"/>
+<part name="J6" library="SparkFun-Connectors" deviceset="QWIIC_CONNECTOR" device="" value="Vertical Qwiic Connector"/>
 </parts>
 <sheets>
@@
 <attribute name="VALUE" x="226.06" y="170.434" size="1.778" layer="96" align="bottom-center"/>
 </instance>
+<instance part="GND5" gate="1" x="218.44" y="88.9" smashed="yes">
+<attribute name="VALUE" x="218.44" y="88.646" size="1.778" layer="96" align="top-center"/>
+</instance>
+<instance part="SUPPLY6" gate="G$1" x="220.98" y="109.22" smashed="yes">
+<attribute name="VALUE" x="220.98" y="112.014" size="1.778" layer="96" align="bottom-center"/>
+</instance>
+<instance part="J2" gate="G$1" x="137.16" y="154.94" smashed="yes">
+<attribute name="VALUE" x="134.62" y="150.114" size="1.778" layer="96" font="vector"/>
+<attribute name="NAME" x="134.62" y="160.528" size="1.778" layer="95" font="vector"/>
+</instance>
+<instance part="F1" gate="F1" x="40.64" y="109.22" smashed="yes">
+<attribute name="NAME" x="35.687" y="117.221" size="1.778" layer="95" font="vector" rot="R180" align="bottom-center"/>
+<attribute name="VALUE" x="41.91" y="112.014" size="2.286" layer="96" font="vector" rot="R180" align="top-center"/>
+</instance>
+<instance part="JP1" gate="G$1" x="43.18" y="99.06" smashed="yes">
+<attribute name="NAME" x="45.466" y="101.854" size="1.778" layer="95" font="vector"/>
+</instance>
+<instance part="LOGO3" gate="G$1" x="187.96" y="33.02" smashed="yes"/>
 <instance part="J5" gate="G$1" x="172.72" y="76.2" smashed="yes" rot="MR180">
 <attribute name="VALUE" x="167.64" y="81.534" size="1.778" layer="96" font="vector" rot="MR180" align="top-left"/>
@@
 <attribute name="NAME" x="203.2" y="93.726" size="1.778" layer="95" font="vector" rot="MR180"/>
 </instance>
-<instance part="GND5" gate="1" x="218.44" y="88.9" smashed="yes">
-<attribute name="VALUE" x="218.44" y="88.646" size="1.778" layer="96" align="top-center"/>
-</instance>
-<instance part="SUPPLY6" gate="G$1" x="220.98" y="109.22" smashed="yes">
-<attribute name="VALUE" x="220.98" y="112.014" size="1.778" layer="96" align="bottom-center"/>
-</instance>
-<instance part="J2" gate="G$1" x="137.16" y="154.94" smashed="yes">
-<attribute name="VALUE" x="134.62" y="150.114" size="1.778" layer="96" font="vector"/>
-<attribute name="NAME" x="134.62" y="160.528" size="1.778" layer="95" font="vector"/>
-</instance>
-<instance part="F1" gate="F1" x="40.64" y="109.22" smashed="yes">
-<attribute name="NAME" x="35.687" y="117.221" size="1.778" layer="95" font="vector" rot="R180" align="bottom-center"/>
-<attribute name="VALUE" x="41.91" y="112.014" size="2.286" layer="96" font="vector" rot="R180" align="top-center"/>
-</instance>
-<instance part="JP1" gate="G$1" x="43.18" y="99.06" smashed="yes">
-<attribute name="NAME" x="45.466" y="101.854" size="1.778" layer="95" font="vector"/>
-</instance>
-<instance part="LOGO3" gate="G$1" x="187.96" y="33.02" smashed="yes"/>
 </instances>
 <busses>
@@
 <wire x1="180.34" y1="104.14" x2="182.88" y2="104.14" width="0.1524" layer="91"/>
 <wire x1="182.88" y1="104.14" x2="182.88" y2="78.74" width="0.1524" layer="91"/>
-<pinref part="J5" gate="G$1" pin="1"/>
 <wire x1="182.88" y1="78.74" x2="182.88" y2="66.04" width="0.1524" layer="91"/>
 <wire x1="180.34" y1="78.74" x2="182.88" y2="78.74" width="0.1524" layer="91"/>
 <junction x="182.88" y="78.74"/>
+<pinref part="J5" gate="G$1" pin="1"/>
 </segment>
 <segment>
@@
 <wire x1="38.1" y1="53.34" x2="35.56" y2="53.34" width="0.1524" layer="91"/>
 <wire x1="35.56" y1="53.34" x2="35.56" y2="50.8" width="0.1524" layer="91"/>
-<pinref part="J1" gate="G$1" pin="GND@9"/>
 <wire x1="35.56" y1="50.8" x2="35.56" y2="48.26" width="0.1524" layer="91"/>
 <wire x1="35.56" y1="48.26" x2="35.56" y2="45.72" width="0.1524" layer="91"/>
@@
 <wire x1="35.56" y1="38.1" x2="35.56" y2="35.56" width="0.1524" layer="91"/>
 <wire x1="35.56" y1="35.56" x2="35.56" y2="27.94" width="0.1524" layer="91"/>
-<wire x1="38.1" y1="50.8" x2="35.56" y2="50.8" width="0.1524" layer="91"/>
-<junction x="35.56" y="50.8"/>
 <pinref part="J1" gate="G$1" pin="GND@14"/>
 <wire x1="38.1" y1="48.26" x2="35.56" y2="48.26" width="0.1524" layer="91"/>
@@
 <junction x="35.56" y="35.56"/>
 <pinref part="GND1" gate="1" pin="GND"/>
+<pinref part="J1" gate="G$1" pin="GND@9"/>
+<wire x1="38.1" y1="50.8" x2="35.56" y2="50.8" width="0.1524" layer="91"/>
+<junction x="35.56" y="50.8"/>
 </segment>
 <segment>
@@
 </segment>
 <segment>
-<pinref part="J6" gate="G$1" pin="1"/>
 <wire x1="215.9" y1="104.14" x2="218.44" y2="104.14" width="0.1524" layer="91"/>
 <wire x1="218.44" y1="104.14" x2="218.44" y2="91.44" width="0.1524" layer="91"/>
 <pinref part="GND5" gate="1" pin="GND"/>
+<pinref part="J6" gate="G$1" pin="1"/>
 </segment>
 <segment>
@@
 <wire x1="185.42" y1="101.6" x2="185.42" y2="109.22" width="0.1524" layer="91"/>
 <pinref part="SUPPLY5" gate="G$1" pin="3.3V"/>
-<pinref part="J5" gate="G$1" pin="2"/>
 <wire x1="180.34" y1="76.2" x2="185.42" y2="76.2" width="0.1524" layer="91"/>
 <wire x1="185.42" y1="76.2" x2="185.42" y2="101.6" width="0.1524" layer="91"/>
 <junction x="185.42" y="101.6"/>
+<pinref part="J5" gate="G$1" pin="2"/>
 </segment>
 <segment>
@@
 </segment>
 <segment>
-<pinref part="J6" gate="G$1" pin="2"/>
 <wire x1="215.9" y1="101.6" x2="220.98" y2="101.6" width="0.1524" layer="91"/>
 <wire x1="220.98" y1="101.6" x2="220.98" y2="109.22" width="0.1524" layer="91"/>
@@
 <wire x1="220.98" y1="73.66" x2="220.98" y2="101.6" width="0.1524" layer="91"/>
 <junction x="220.98" y="101.6"/>
+<pinref part="J6" gate="G$1" pin="2"/>
 </segment>
 </net>
@@
 </segment>
 <segment>
-<pinref part="J5" gate="G$1" pin="3"/>
 <wire x1="180.34" y1="73.66" x2="185.42" y2="73.66" width="0.1524" layer="91"/>
 <label x="185.42" y="73.66" size="1.27" layer="95" xref="yes"/>
-</segment>
-<segment>
-<pinref part="J6" gate="G$1" pin="3"/>
+<pinref part="J5" gate="G$1" pin="3"/>
+</segment>
+<segment>
 <wire x1="215.9" y1="99.06" x2="223.52" y2="99.06" width="0.1524" layer="91"/>
 <label x="223.52" y="99.06" size="1.27" layer="95" xref="yes"/>
+<pinref part="J6" gate="G$1" pin="3"/>
 </segment>
 </net>
@@
 </segment>
 <segment>
-<pinref part="J5" gate="G$1" pin="4"/>
 <wire x1="180.34" y1="71.12" x2="185.42" y2="71.12" width="0.1524" layer="91"/>
 <label x="185.42" y="71.12" size="1.27" layer="95" xref="yes"/>
-</segment>
-<segment>
-<pinref part="J6" gate="G$1" pin="4"/>
+<pinref part="J5" gate="G$1" pin="4"/>
+</segment>
+<segment>
 <wire x1="215.9" y1="96.52" x2="223.52" y2="96.52" width="0.1524" layer="91"/>
 <label x="223.52" y="96.52" size="1.27" layer="95" xref="yes"/>
+<pinref part="J6" gate="G$1" pin="4"/>
 </segment>
 </net>
@@
 <pinref part="R2" gate="G$1" pin="2"/>
 <wire x1="60.96" y1="147.32" x2="58.42" y2="147.32" width="0.1524" layer="91"/>
-</segment>
-</net>
-<net name="N$1" class="0">
-<segment>
-<pinref part="J1" gate="G$1" pin="3.3V@1"/>
-<wire x1="38.1" y1="86.36" x2="35.56" y2="86.36" width="0.1524" layer="91"/>
 </segment>
 </net>
@@
 </segment>
 </net>
+<net name="N$1" class="0">
+<segment>
+<pinref part="J1" gate="G$1" pin="3.3V@1"/>
+<wire x1="38.1" y1="86.36" x2="35.56" y2="86.36" width="0.1524" layer="91"/>
+</segment>
+</net>
