File: Production/Qwiic_pHat_for_Raspberry_Pi_v30-Panel.brd (EAGLE design)
At the start: 85.1 x 174.6 mm, 228 parts, among them J1 RASPBERRYPI-40-PIN-GPIO_PTH_N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, J10 RASPBERRYPI-40-PIN-GPIO_PTH_N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, J15 Qwiic Right Angle, J16 Qwiic Right Angle, J17 RASPBERRYPI-40-PIN-GPIO_PTH_N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, J22 Qwiic Right Angle, J23 Qwiic Right Angle, J24 RASPBERRYPI-40-PIN-GPIO_PTH_N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, J29 Qwiic Right Angle, J30 Qwiic Right Angle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

Commit message: Adds updated production panel
Parts:
- removed U$81, U$84: (no value), POWER:5V0
- removed U$82, U$83: (no value), POWER:POWER1
- removed U$85, U$86, U$87: (no value), SparkFun-Aesthetics:QWIIC_3MM
- removed U$88: (no value), Qwiic:QWIIC0
- removed U$89: (no value), pie_1f967#png:PIE_1F967#PNG
- removed U$90: (no value), SparkFun-Aesthetics:SFE_LOGO_NAME_FLAME_.3
- added FRAME1, FRAME2, FRAME3, FRAME4, FRAME5: FRAME-LETTER, SparkFun-Aesthetics:CREATIVE_COMMONS
- J12, J19, J26, J33: device SparkFun-Connectors:JST04_1MM_VERT -> SparkFun-Connectors:SCREWTERMINAL-3.5MM-2-NS
- J13, J20, J27, J34, J5, J6: value (none) -> Vertical Qwiic Connector
- J14, J21, J28, J35: value (none) -> Vertical Qwiic Connector; device SparkFun-Connectors:SCREWTERMINAL-3.5MM-2-NS -> SparkFun-Connectors:JST04_1MM_VERT
- U$19: device MicroPiHat:PHAT0 -> All labels:GPIO173
- U$20: device Labels:I2C-() -> Fuse Bypass:FUSE0
- U$21: device SparkX:QWIIC_BOARD_MOUNT_NOHOLES -> Fuse Bypass:BYPASS1
- U$22, U$75, U$76: device SparkX:QWIIC_BOARD_MOUNT_NOHOLES -> SparkFun-Aesthetics:QWIIC_3MM
- U$23: device All labels:GPIO173 -> POWER:5V0
- U$24: device Fuse Bypass:FUSE0 -> POWER:POWER1
- U$25: device Fuse Bypass:BYPASS1 -> POWER:POWER1
- U$26: device SparkFun-Aesthetics:QWIIC_3MM -> POWER:5V0
- U$27, U$45: device POWER:5V0 -> SparkFun-Aesthetics:QWIIC_3MM
- U$28, U$29: device POWER:POWER1 -> SparkFun-Aesthetics:QWIIC_3MM
- U$30: device POWER:5V0 -> Qwiic:QWIIC0
- U$31: device SparkFun-Aesthetics:QWIIC_3MM -> pie_1f967#png:PIE_1F967#PNG
- U$32, U$80: device SparkFun-Aesthetics:QWIIC_3MM -> SparkFun-Aesthetics:SFE_LOGO_NAME_FLAME_.3
- U$33, U$49: device SparkFun-Aesthetics:QWIIC_3MM -> MicroPiHat:PHAT0
- U$34: device Qwiic:QWIIC0 -> Labels:I2C-()
- U$35: device pie_1f967#png:PIE_1F967#PNG -> All labels:GPIO173
- U$36: device SparkFun-Aesthetics:SFE_LOGO_NAME_FLAME_.3 -> Fuse Bypass:FUSE0
- U$37: device MicroPiHat:PHAT0 -> Fuse Bypass:BYPASS1
- U$38: device Labels:I2C-() -> SparkFun-Aesthetics:QWIIC_3MM
- U$39, U$58: device SparkX:QWIIC_BOARD_MOUNT_NOHOLES -> POWER:5V0
- U$4: device SparkX:QWIIC_BOARD_MOUNT_NOHOLES -> MicroPiHat:PHAT0
- U$40, U$57: device SparkX:QWIIC_BOARD_MOUNT_NOHOLES -> POWER:POWER1
- U$41: device All labels:GPIO173 -> POWER:POWER1
- U$42: device Fuse Bypass:FUSE0 -> POWER:5V0
- U$43, U$61: device Fuse Bypass:BYPASS1 -> SparkFun-Aesthetics:QWIIC_3MM
- U$46: device POWER:POWER1 -> Qwiic:QWIIC0
- U$47: device POWER:POWER1 -> pie_1f967#png:PIE_1F967#PNG
- U$48: device POWER:5V0 -> SparkFun-Aesthetics:SFE_LOGO_NAME_FLAME_.3
- U$5: device SparkX:QWIIC_BOARD_MOUNT_NOHOLES -> Labels:I2C-()
- U$50: device SparkFun-Aesthetics:QWIIC_3MM -> Labels:I2C-()
- U$51, U$67: device SparkFun-Aesthetics:QWIIC_3MM -> All labels:GPIO173
- U$52: device Qwiic:QWIIC0 -> Fuse Bypass:FUSE0
- U$53: device pie_1f967#png:PIE_1F967#PNG -> Fuse Bypass:BYPASS1
- U$54: device SparkFun-Aesthetics:SFE_LOGO_NAME_FLAME_.3 -> SparkFun-Aesthetics:QWIIC_3MM
- U$55: device MicroPiHat:PHAT0 -> POWER:5V0
- U$56: device Labels:I2C-() -> POWER:POWER1
- U$59, U$77: device All labels:GPIO173 -> SparkFun-Aesthetics:QWIIC_3MM
- U$60: device Fuse Bypass:FUSE0 -> SparkFun-Aesthetics:QWIIC_3MM
- U$62: device SparkFun-Aesthetics:QWIIC_3MM -> Qwiic:QWIIC0
- U$63: device POWER:5V0 -> pie_1f967#png:PIE_1F967#PNG
- U$64: device POWER:POWER1 -> SparkFun-Aesthetics:SFE_LOGO_NAME_FLAME_.3
- U$65: device POWER:POWER1 -> MicroPiHat:PHAT0
- U$66: device POWER:5V0 -> Labels:I2C-()
- U$68: device SparkFun-Aesthetics:QWIIC_3MM -> Fuse Bypass:FUSE0
- U$69: device SparkFun-Aesthetics:QWIIC_3MM -> Fuse Bypass:BYPASS1
- U$70: device Qwiic:QWIIC0 -> SparkFun-Aesthetics:QWIIC_3MM
- U$71: device pie_1f967#png:PIE_1F967#PNG -> POWER:5V0
- U$72: device SparkFun-Aesthetics:SFE_LOGO_NAME_FLAME_.3 -> POWER:POWER1
- U$73: device MicroPiHat:PHAT0 -> POWER:POWER1
- U$74: device Labels:I2C-() -> POWER:5V0
- U$78: device Fuse Bypass:FUSE0 -> Qwiic:QWIIC0
- U$79: device Fuse Bypass:BYPASS1 -> pie_1f967#png:PIE_1F967#PNG
- moved U$70 67.4 mm to (63.0, 147.4)
- moved U$5 65.1 mm to (13.3, 46.1)
- moved U$27 64.3 mm to (63.2, 45.7)
- moved U$26 58.7 mm to (5.33, 43.5), flipped to the bottom
- moved U$40 55.0 mm to (-1.02, 72.2)
- moved U$75 54.0 mm to (63.2, 138.8)
- moved U$54 52.1 mm to (63.0, 116.4), flipped to the top
- moved U$62 51.8 mm to (13.2, 101.9)
- moved U$38 50.4 mm to (63.0, 85.4)
- moved U$58 49.8 mm to (5.33, 105.5), flipped to the bottom
- moved U$4 49.8 mm to (30.3, 40.2)
- moved U$43 47.4 mm to (63.2, 76.7), flipped to the top
- moved U$23 46.6 mm to (-1.02, 43.5)
- moved U$36 46.4 mm to (14.2, 84.6)
- moved U$72 45.6 mm to (-1.02, 134.2), flipped to the top
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Connections:
- net 3.3V1: now also J14.2; no longer J12.2
- net 3.3V2: now also J21.2; no longer J19.2
- net 3.3V3: now also J28.2; no longer J26.2
- net 3.3V4: now also J35.2; no longer J33.2
- net 5V1: now also J12.2; no longer J14.2
- net 5V2: now also J19.2; no longer J21.2
- net 5V3: now also J26.2; no longer J28.2
- net 5V4: now also J33.2; no longer J35.2
- net SCL1: now also J14.4; no longer J12.4
- net SCL2: now also J21.4; no longer J19.4
- net SCL3: now also J28.4; no longer J26.4
- net SCL4: now also J35.4; no longer J33.4
- net SDA1: now also J14.3; no longer J12.3
- net SDA2: now also J21.3; no longer J19.3
- net SDA3: now also J28.3; no longer J26.3
- net SDA4: now also J35.3; no longer J33.3
